Commit message: ALLEX Model v0.1.2

File: urdf/ALLEX.urdf (robot description, URDF)
Before this commit: robot ALLEX, 72 links, 71 joints
Links:
- link Base_Link: mass 3 -> 3.0
- link Chest_Origin_Link: mass 0 -> 0.0
- link L_Palm_Link: mass 0.553111 -> 0.0
- link L_Wrist_Pitch_Link: mass 1.025201999 -> 0.767755918
- link R_Palm_Link: mass 0.553111 -> 0.0
- link R_Wrist_Pitch_Link: mass 1.025201999 -> 0.767755918

Commit message: Republish from SSoT proto_v2 (repo renamed allex_description → allex_model)
- repo renamed: allex_description → allex_model
- USD: fix drive kp unit conversion (deg→rad) — emit_usd bug fix, now in published USD
- MJCF (ALLEX.xml): drop velocity/effort limits comment (info is in URDF <limit> + sidecar)
- regenerated URDF/MJCF/USD + flattened mesh from allex/model (launch/rviz preserved)

File: urdf/ALLEX.urdf (robot description, URDF)
Before this commit: robot ALLEX, 82 links, 81 joints
Links:
- link Base_Link: mass 3.0 -> 3
- link Chest_Origin_Link: mass 0.0 -> 0
- link L_Forearm_Link: mass 3.026739291 -> 3.02673929
- link L_Palm_Link: mass 0.0 -> 0
- link L_Shoulder_Pitch_Link: mass 1.015421884 -> 1.01542188
- link L_Shoulder_RollYaw_Link: mass 2.869014517 -> 2.86901452
- link Neck_Yaw_Link: mass 1.884994309 -> 1.88499431
- link R_Forearm_Link: mass 3.026739291 -> 3.02673929
- link R_Palm_Link: mass 0.0 -> 0
- link R_Shoulder_Pitch_Link: mass 1.015421884 -> 1.01542188
- link R_Shoulder_RollYaw_Link: mass 2.869014517 -> 2.86901452
- link Waist_Upper_Pitch_Link: mass 3.247447863 -> 3.24744786
Joints:
- removed joint Chest_Origin_fixed_Joint
- removed joint L_Index_Fingertip_Joint
- removed joint L_Little_Fingertip_Joint
- removed joint L_Middle_Fingertip_Joint
- removed joint L_Palm_fixed_Joint
- removed joint L_Ring_Fingertip_Joint
- removed joint L_Thumb_Fingertip_Joint
- removed joint R_Index_Fingertip_Joint
- removed joint R_Little_Fingertip_Joint
- removed joint R_Middle_Fingertip_Joint
- removed joint R_Palm_fixed_Joint
- removed joint R_Ring_Fingertip_Joint
- removed joint R_Thumb_Fingertip_Joint
- removed joint orbbec_link_fixed_Joint
- removed joint realsense_link_fixed_Joint
- removed joint zed_camera_link_fixed_Joint
- added joint Chest_Origin_Link_fixed_joint: type fixed, parent Waist_Upper_Pitch_Link, child Chest_Origin_Link, origin xyz=0.0415 0 0.149 rpy=0 0 0
- added joint L_Index_Fingertip_fixed_joint: type fixed, parent L_Index_Distal_Link, child L_Index_Fingertip, origin xyz=0.0075 0 -0.011 rpy=0 0 0
- added joint L_Little_Fingertip_fixed_joint: type fixed, parent L_Little_Distal_Link, child L_Little_Fingertip, origin xyz=0.0075 0 -0.011 rpy=0 0 0
- added joint L_Middle_Fingertip_fixed_joint: type fixed, parent L_Middle_Distal_Link, child L_Middle_Fingertip, origin xyz=0.0075 0 -0.011 rpy=0 0 0
- added joint L_Palm_Link_fixed_joint: type fixed, parent L_Wrist_Pitch_Link, child L_Palm_Link, origin xyz=0.0045 0 -0.095 rpy=0 0 0
- added joint L_Ring_Fingertip_fixed_joint: type fixed, parent L_Ring_Distal_Link, child L_Ring_Fingertip, origin xyz=0.0075 0 -0.011 rpy=0 0 0
- added joint L_Thumb_Fingertip_fixed_joint: type fixed, parent L_Thumb_Distal_Link, child L_Thumb_Fingertip, origin xyz=0 0.011 -0.006 rpy=0 0 0
- added joint R_Index_Fingertip_fixed_joint: type fixed, parent R_Index_Distal_Link, child R_Index_Fingertip, origin xyz=0.0075 0 -0.011 rpy=0 0 0
- added joint R_Little_Fingertip_fixed_joint: type fixed, parent R_Little_Distal_Link, child R_Little_Fingertip, origin xyz=0.0075 0 -0.011 rpy=0 0 0
- added joint R_Middle_Fingertip_fixed_joint: type fixed, parent R_Middle_Distal_Link, child R_Middle_Fingertip, origin xyz=0.0075 0 -0.011 rpy=0 0 0
- added joint R_Palm_Link_fixed_joint: type fixed, parent R_Wrist_Pitch_Link, child R_Palm_Link, origin xyz=0.0045 0 -0.095 rpy=0 0 0
- added joint R_Ring_Fingertip_fixed_joint: type fixed, parent R_Ring_Distal_Link, child R_Ring_Fingertip, origin xyz=0.0075 0 -0.011 rpy=0 0 0
- added joint R_Thumb_Fingertip_fixed_joint: type fixed, parent R_Thumb_Distal_Link, child R_Thumb_Fingertip, origin xyz=0 -0.011 -0.006 rpy=0 0 0
- added joint orbbec_link_fixed_joint: type fixed, parent Neck_Yaw_Link, child orbbec_link, origin xyz=0.0893 0.002 0.0733 rpy=0 0 0
- added joint realsense_link_fixed_joint: type fixed, parent Neck_Yaw_Link, child realsense_link, origin xyz=0.0753 0 0.1029 rpy=0 0 0
- added joint zed_camera_link_fixed_joint: type fixed, parent Neck_Yaw_Link, child zed_camera_link, origin xyz=0.067225 0 0.0145 rpy=0 0 0
- joint L_Index_ABAD_Joint: origin xyz=-0.0186259 0.0330567 -0.0383928 rpy=0.11155943312272709 -0.34233803538908836 -0.0870605140350752 -> xyz=-0.0186259 0.0330567 -0.0383928 rpy=0.111559433 -0.342338035 -0.087060514
- joint L_Index_DIP_Joint: limit lower=0 upper=1.235693 effort=3 velocity=10 -> lower=0 upper=1.10975556 effort=3 velocity=10; mimic joint=L_Index_PIP_Joint multiplier=0.6361 offset=0 -> joint=L_Index_PIP_Joint multiplier=0.635843082 offset=0
- joint L_Index_MCP_Joint: origin xyz=-0.003817 0 -0.0061246 rpy=0 0.3490658780677358 0 -> xyz=-0.003817 0 -0.0061246 rpy=0 0.349065878 0
- joint L_Little_ABAD_Joint: origin xyz=-0.0185852 -0.0327196 -0.0383938 rpy=-0.22099136278843234 -0.3223829827602436 0.1716472165028659 -> xyz=-0.0185852 -0.0327196 -0.0383938 rpy=-0.220991363 -0.322382983 0.171647217
- joint L_Little_DIP_Joint: limit lower=0 upper=1.235693 effort=3 velocity=10 -> lower=0 upper=1.10975556 effort=3 velocity=10; mimic joint=L_Little_PIP_Joint multiplier=0.6361 offset=0 -> joint=L_Little_PIP_Joint multiplier=0.635843082 offset=0
- joint L_Little_MCP_Joint: origin xyz=-0.003817 0 -0.0061246 rpy=0 0.3490658780677358 0 -> xyz=-0.003817 0 -0.0061246 rpy=0 0.349065878 0
- joint L_Middle_ABAD_Joint: origin xyz=-0.0197378 0.0111686 -0.0403088 rpy=0 -0.3490658780677358 0 -> xyz=-0.0197378 0.0111686 -0.0403088 rpy=0 -0.349065878 0
- joint L_Middle_DIP_Joint: limit lower=0 upper=1.235693 effort=3 velocity=10 -> lower=0 upper=1.10975556 effort=3 velocity=10; mimic joint=L_Middle_PIP_Joint multiplier=0.6361 offset=0 -> joint=L_Middle_PIP_Joint multiplier=0.635843082 offset=0
- joint L_Middle_MCP_Joint: origin xyz=-0.003817 0 -0.0061246 rpy=0 0.3490658780677358 0 -> xyz=-0.003817 0 -0.0061246 rpy=0 0.349065878 0
- joint L_Ring_ABAD_Joint: origin xyz=-0.0197763 -0.0108314 -0.0403090 rpy=-0.11155943312272709 -0.34233803538908836 0.0870605140350752 -> xyz=-0.0197763 -0.0108314 -0.040309 rpy=-0.111559433 -0.342338035 0.087060514
- joint L_Ring_DIP_Joint: limit lower=0 upper=1.235693 effort=3 velocity=10 -> lower=0 upper=1.10975556 effort=3 velocity=10; mimic joint=L_Ring_PIP_Joint multiplier=0.6361 offset=0 -> joint=L_Ring_PIP_Joint multiplier=0.635843082 offset=0
- joint L_Ring_MCP_Joint: origin xyz=-0.003817 0 -0.0061246 rpy=0 0.3490658780677358 0 -> xyz=-0.003817 0 -0.0061246 rpy=0 0.349065878 0
- joint L_Shoulder_Pitch_Joint: origin xyz=0 0.0710988 0.0190509 rpy=0.2617993931425453 5.720983553558767e-08 2.6299670132234887e-06 -> xyz=0 0.0710988 0.0190509 rpy=0.261799393 5.72098355e-08 2.62996701e-06
- joint L_Shoulder_Roll_Joint: origin xyz=-0.1365 0.1195 0 rpy=-0.2617993931425453 -5.720983531354307e-08 2.6299670132234887e-06 -> xyz=-0.1365 0.1195 0 rpy=-0.261799393 -5.72098353e-08 2.62996701e-06
- joint L_Thumb_CMC_Joint: origin xyz=0 0.0139985 -0.0323434 rpy=-0.268480430783685 0 0 -> xyz=0 0.0139985 -0.0323434 rpy=-0.268480431 0 0
- joint L_Thumb_IP_Joint: limit lower=0 upper=1.1397 effort=4.8 velocity=8 -> lower=0 upper=1.14964202 effort=4.8 velocity=8; mimic joint=L_Thumb_MCP_Joint multiplier=0.7319 offset=0 -> joint=L_Thumb_MCP_Joint multiplier=0.731884995 offset=0
- joint L_Thumb_Yaw_Joint: origin xyz=0.0098274 0.0210533 0.0360908 rpy=0.08570131975411865 0.12731092045638293 -0.1266080083114749 -> xyz=0.0098274 0.0210533 0.0360908 rpy=0.0857013198 0.12731092 -0.126608008
- joint R_Index_ABAD_Joint: origin xyz=-0.0186259 -0.0330567 -0.0383928 rpy=-0.11155943312272709 -0.34233803538908836 0.0870605140350752 -> xyz=-0.0186259 -0.0330567 -0.0383928 rpy=-0.111559433 -0.342338035 0.087060514
- joint R_Index_DIP_Joint: limit lower=0 upper=1.235693 effort=3 velocity=10 -> lower=0 upper=1.10975556 effort=3 velocity=10; mimic joint=R_Index_PIP_Joint multiplier=0.6361 offset=0 -> joint=R_Index_PIP_Joint multiplier=0.635843082 offset=0
- joint R_Index_MCP_Joint: origin xyz=-0.003817 0 -0.0061246 rpy=0 0.3490658780677358 0 -> xyz=-0.003817 0 -0.0061246 rpy=0 0.349065878 0
- joint R_Little_ABAD_Joint: origin xyz=-0.0185852 0.0327196 -0.0383938 rpy=0.22099136278843234 -0.3223829827602436 -0.1716472165028659 -> xyz=-0.0185852 0.0327196 -0.0383938 rpy=0.220991363 -0.322382983 -0.171647217
- joint R_Little_DIP_Joint: limit lower=0 upper=1.235693 effort=3 velocity=10 -> lower=0 upper=1.10975556 effort=3 velocity=10; mimic joint=R_Little_PIP_Joint multiplier=0.6361 offset=0 -> joint=R_Little_PIP_Joint multiplier=0.635843082 offset=0
- joint R_Little_MCP_Joint: origin xyz=-0.003817 0 -0.0061246 rpy=0 0.3490658780677358 0 -> xyz=-0.003817 0 -0.0061246 rpy=0 0.349065878 0
- joint R_Middle_ABAD_Joint: origin xyz=-0.0197378 -0.0111686 -0.0403088 rpy=0 -0.3490658780677358 0 -> xyz=-0.0197378 -0.0111686 -0.0403088 rpy=0 -0.349065878 0
- joint R_Middle_DIP_Joint: limit lower=0 upper=1.235693 effort=3 velocity=10 -> lower=0 upper=1.10975556 effort=3 velocity=10; mimic joint=R_Middle_PIP_Joint multiplier=0.6361 offset=0 -> joint=R_Middle_PIP_Joint multiplier=0.635843082 offset=0
- joint R_Middle_MCP_Joint: origin xyz=-0.003817 0 -0.0061246 rpy=0 0.3490658780677358 0 -> xyz=-0.003817 0 -0.0061246 rpy=0 0.349065878 0
- joint R_Ring_ABAD_Joint: origin xyz=-0.0197763 0.0108314 -0.0403090 rpy=0.11155943312272709 -0.34233803538908836 -0.0870605140350752 -> xyz=-0.0197763 0.0108314 -0.040309 rpy=0.111559433 -0.342338035 -0.087060514
- joint R_Ring_DIP_Joint: limit lower=0 upper=1.235693 effort=3 velocity=10 -> lower=0 upper=1.10975556 effort=3 velocity=10; mimic joint=R_Ring_PIP_Joint multiplier=0.6361 offset=0 -> joint=R_Ring_PIP_Joint multiplier=0.635843082 offset=0
- joint R_Ring_MCP_Joint: origin xyz=-0.003817 0 -0.0061246 rpy=0 0.3490658780677358 0 -> xyz=-0.003817 0 -0.0061246 rpy=0 0.349065878 0
- joint R_Shoulder_Pitch_Joint: origin xyz=0 -0.0710988 0.0190509 rpy=-0.2617993931425453 -5.720983531354307e-08 2.6299670132234887e-06 -> xyz=0 -0.0710988 0.0190509 rpy=-0.261799393 -5.72098353e-08 2.62996701e-06
- joint R_Shoulder_Roll_Joint: origin xyz=-0.1365 -0.1195 0 rpy=0.2617993931425453 5.720983553558767e-08 2.6299670132234887e-06 -> xyz=-0.1365 -0.1195 0 rpy=0.261799393 5.72098355e-08 2.62996701e-06
- joint R_Thumb_CMC_Joint: origin xyz=0 -0.0139985 -0.0323434 rpy=0.268480430783685 0 0 -> xyz=0 -0.0139985 -0.0323434 rpy=0.268480431 0 0
- joint R_Thumb_IP_Joint: limit lower=0 upper=1.1397 effort=4.8 velocity=8 -> lower=0 upper=1.14964202 effort=4.8 velocity=8; mimic joint=R_Thumb_MCP_Joint multiplier=0.7319 offset=0 -> joint=R_Thumb_MCP_Joint multiplier=0.731884995 offset=0
- joint R_Thumb_Yaw_Joint: origin xyz=0.0098263 -0.0210097 0.0360889 rpy=-0.08570131975411865 0.12731092045638293 0.1266080083114749 -> xyz=0.0098263 -0.0210097 0.0360889 rpy=-0.0857013198 0.12731092 0.126608008
- joint orbbec_color_optical_frame_joint: origin xyz=-0.002 -0.033 -0.001 rpy=0 1.5708 0 -> xyz=-0.002 -0.033 -0.001 rpy=-0 1.57079633 0
- joint orbbec_depth_optical_frame_joint: origin xyz=0 0 0 rpy=0 1.5708 0 -> xyz=0 0 0 rpy=-0 1.57079633 0
- joint realsense_color_optical_frame_joint: origin xyz=0.011 0.033 0.013 rpy=0 1.5708 0 -> xyz=0.011 0.033 0.013 rpy=-0 1.57079633 0
- joint realsense_depth_optical_frame_joint: origin xyz=0.011 0.018 0.013 rpy=0 1.5708 0 -> xyz=0.011 0.018 0.013 rpy=-0 1.57079633 0
- joint zed_left_camera_optical_frame_joint: origin xyz=0 0.032 0.013 rpy=0 1.5708 0 -> xyz=0 0.032 0.013 rpy=-0 1.57079633 0

Commit message: Republish proto_v1 from SSoT: add USD, regenerate urdf/mjcf
Regenerated from the allex generator (SSoT spec/proto_v1). Adds usd/ALLEX.usd
(46.7MB PhysX base) — proto_v1 previously shipped no USD. Regenerates urdf/mjcf
to the generator's canonical output: physics (mass/inertia/coupling) identical
to the prior v0.1.2, with named equality joints, *_fixed_joint naming, and
L_Middle distal link normalized to L_Middle_Distal_Link. meshes unchanged.

File: urdf/ALLEX.urdf (robot description, URDF)
Before this commit: robot ALLEX, 72 links, 71 joints
Links:
- link Base_Link: mass 3.0 -> 3
- link Chest_Origin_Link: mass 0.0 -> 0
- link L_Palm_Link: mass 0.0 -> 0
- link L_Shoulder_Pitch_Link: mass 1.015421884 -> 1.01542188
- link L_Shoulder_Roll_Link: mass 2.869014517 -> 2.86901452
- link L_Shoulder_Yaw_Link: mass 3.544274792 -> 3.54427479
- link L_Wrist_Yaw_Link: mass 2.626560674 -> 2.62656067
- link Neck_Yaw_Link: mass 1.884994309 -> 1.88499431
- link R_Palm_Link: mass 0.0 -> 0
- link R_Shoulder_Pitch_Link: mass 1.015421884 -> 1.01542188
- link R_Shoulder_Roll_Link: mass 2.869014517 -> 2.86901452
- link R_Shoulder_Yaw_Link: mass 3.544274792 -> 3.54427479
- link R_Wrist_Yaw_Link: mass 2.626560674 -> 2.62656067
- link Waist_Upper_Pitch_Link: mass 3.247447863 -> 3.24744786
Joints:
- removed joint Chest_Origin_fixed_Joint
- removed joint L_Palm_fixed_Joint
- removed joint R_Palm_fixed_Joint
- removed joint orbbec_link_fixed_Joint
- removed joint realsense_link_fixed_Joint
- removed joint zed_camera_link_fixed_Joint
- added joint Chest_Origin_Link_fixed_joint: type fixed, parent Waist_Upper_Pitch_Link, child Chest_Origin_Link, origin xyz=0.0415 0 0.1169196 rpy=0 0 0
- added joint L_Palm_Link_fixed_joint: type fixed, parent L_Wrist_Pitch_Link, child L_Palm_Link, origin xyz=-0.0191006 0.00915 -0.086757 rpy=0.0436182662 0.00114172706 -0.0261550729
- added joint R_Palm_Link_fixed_joint: type fixed, parent R_Wrist_Pitch_Link, child R_Palm_Link, origin xyz=-0.0191006 -0.00915 -0.086757 rpy=-0.0436182662 0.00114172706 0.0261550729
- added joint orbbec_link_fixed_joint: type fixed, parent Neck_Yaw_Link, child orbbec_link, origin xyz=0.0893 0.002 0.0733 rpy=0 0 0
- added joint realsense_link_fixed_joint: type fixed, parent Neck_Yaw_Link, child realsense_link, origin xyz=0.0753 0 0.1029 rpy=0 0 0
- added joint zed_camera_link_fixed_joint: type fixed, parent Neck_Yaw_Link, child zed_camera_link, origin xyz=0.067225 0 0.0145 rpy=0 0 0
- joint L_Index_ABAD_Joint: origin xyz=0.004401 0.0219725 -0.0476342 rpy=0.11155943312272709 -0.34233803538908836 -0.0870605140350752 -> xyz=0.004401 0.0219725 -0.0476342 rpy=0.111559433 -0.342338035 -0.087060514
- joint L_Index_DIP_Joint: limit lower=0 upper=1.235693 effort=3 velocity=10 -> lower=0 upper=1.10975556 effort=0 velocity=0; mimic joint=L_Index_PIP_Joint multiplier=0.6361 offset=0 -> joint=L_Index_PIP_Joint multiplier=0.635843082 offset=0
- joint L_Index_MCP_Joint: origin xyz=-0.003817 0 -0.0061246 rpy=0 0.3490658780677358 0 -> xyz=-0.003817 0 -0.0061246 rpy=0 0.349065878 0
- joint L_Little_ABAD_Joint: origin xyz=0.0061619 -0.0437177 -0.0447661 rpy=-0.22099136278843234 -0.3223829827602436 0.1716472165028659 -> xyz=0.0061619 -0.0437177 -0.0447661 rpy=-0.220991363 -0.322382983 0.171647217
- joint L_Little_DIP_Joint: limit lower=0 upper=1.235693 effort=3 velocity=10 -> lower=0 upper=1.10975556 effort=0 velocity=0; mimic joint=L_Little_PIP_Joint multiplier=0.6361 offset=0 -> joint=L_Little_PIP_Joint multiplier=0.635843082 offset=0
- joint L_Little_MCP_Joint: origin xyz=-0.003817 0 -0.0061246 rpy=0 0.3490658780677358 0 -> xyz=-0.003817 0 -0.0061246 rpy=0 0.349065878 0
- joint L_Middle_ABAD_Joint: origin xyz=0.0038641 0 -0.0485936 rpy=0 -0.3490658780677358 0 -> xyz=0.0038641 0 -0.0485936 rpy=0 -0.349065878 0
- joint L_Middle_DIP_Joint: limit lower=0 upper=1.235693 effort=3 velocity=10 -> lower=0 upper=1.10975556 effort=0 velocity=0; mimic joint=L_Middle_PIP_Joint multiplier=0.6361 offset=0 -> joint=L_Middle_PIP_Joint multiplier=0.635843082 offset=0
- joint L_Middle_MCP_Joint: origin xyz=-0.003817 0 -0.0061246 rpy=0 0.3490658780677358 0 -> xyz=-0.003817 0 -0.0061246 rpy=0 0.349065878 0
- joint L_Ring_ABAD_Joint: origin xyz=0.004401 -0.0219725 -0.0476342 rpy=-0.11155943312272709 -0.34233803538908836 0.0870605140350752 -> xyz=0.004401 -0.0219725 -0.0476342 rpy=-0.111559433 -0.342338035 0.087060514
- joint L_Ring_DIP_Joint: limit lower=0 upper=1.235693 effort=3 velocity=10 -> lower=0 upper=1.10975556 effort=0 velocity=0; mimic joint=L_Ring_PIP_Joint multiplier=0.6361 offset=0 -> joint=L_Ring_PIP_Joint multiplier=0.635843082 offset=0
- joint L_Ring_MCP_Joint: origin xyz=-0.003817 0 -0.0061246 rpy=0 0.3490658780677358 0 -> xyz=-0.003817 0 -0.0061246 rpy=0 0.349065878 0
- joint L_Shoulder_Pitch_Joint: origin xyz=0 0.0710988 0.0190509 rpy=0.2617993931425453 5.720983553558767e-08 2.6299670132234887e-06 -> xyz=0 0.0710988 0.0190509 rpy=0.261799393 5.72098355e-08 2.62996701e-06
- joint L_Shoulder_Roll_Joint: origin xyz=-0.1365 0.1195 0 rpy=-0.2617993931425453 -5.720983531354307e-08 2.6299670132234887e-06 -> xyz=-0.1365 0.1195 0 rpy=-0.261799393 -5.72098353e-08 2.62996701e-06
- joint L_Thumb_CMC_Joint: origin xyz=0 0.0139985 -0.0323434 rpy=-0.268480430783685 0 0 -> xyz=0 0.0139985 -0.0323434 rpy=-0.268480431 0 0
- joint L_Thumb_IP_Joint: limit lower=0 upper=1.1397 effort=4.8 velocity=8 -> lower=0 upper=1.14964202 effort=0 velocity=0; mimic joint=L_Thumb_MCP_Joint multiplier=0.7319 offset=0 -> joint=L_Thumb_MCP_Joint multiplier=0.731884995 offset=0
- joint L_Thumb_Yaw_Joint: origin xyz=0.0330735 0.0139772 0.0273021 rpy=0.08570131975411865 0.12731092045638293 -0.1266080083114749 -> xyz=0.0330735 0.0139772 0.0273021 rpy=0.0857013198 0.12731092 -0.126608008
- joint R_Index_ABAD_Joint: origin xyz=0.004401 -0.0219725 -0.0476342 rpy=-0.11155943312272709 -0.34233803538908836 0.0870605140350752 -> xyz=0.004401 -0.0219725 -0.0476342 rpy=-0.111559433 -0.342338035 0.087060514
- joint R_Index_DIP_Joint: limit lower=0 upper=1.235693 effort=3 velocity=10 -> lower=0 upper=1.10975556 effort=0 velocity=0; mimic joint=R_Index_PIP_Joint multiplier=0.6361 offset=0 -> joint=R_Index_PIP_Joint multiplier=0.635843082 offset=0
- joint R_Index_MCP_Joint: origin xyz=-0.003817 0 -0.0061246 rpy=0 0.3490658780677358 0 -> xyz=-0.003817 0 -0.0061246 rpy=0 0.349065878 0
- joint R_Little_ABAD_Joint: origin xyz=0.0061619 0.0437177 -0.0447661 rpy=0.22099136278843234 -0.3223829827602436 -0.1716472165028659 -> xyz=0.0061619 0.0437177 -0.0447661 rpy=0.220991363 -0.322382983 -0.171647217
- joint R_Little_DIP_Joint: limit lower=0 upper=1.235693 effort=3 velocity=10 -> lower=0 upper=1.10975556 effort=0 velocity=0; mimic joint=R_Little_PIP_Joint multiplier=0.6361 offset=0 -> joint=R_Little_PIP_Joint multiplier=0.635843082 offset=0
- joint R_Little_MCP_Joint: origin xyz=-0.003817 0 -0.0061246 rpy=0 0.3490658780677358 0 -> xyz=-0.003817 0 -0.0061246 rpy=0 0.349065878 0
- joint R_Middle_ABAD_Joint: origin xyz=0.0038641 0 -0.0485936 rpy=0 -0.3490658780677358 0 -> xyz=0.0038641 0 -0.0485936 rpy=0 -0.349065878 0
- joint R_Middle_DIP_Joint: limit lower=0 upper=1.235693 effort=3 velocity=10 -> lower=0 upper=1.10975556 effort=0 velocity=0; mimic joint=R_Middle_PIP_Joint multiplier=0.6361 offset=0 -> joint=R_Middle_PIP_Joint multiplier=0.635843082 offset=0
- joint R_Middle_MCP_Joint: origin xyz=-0.003817 0 -0.0061246 rpy=0 0.3490658780677358 0 -> xyz=-0.003817 0 -0.0061246 rpy=0 0.349065878 0
- joint R_Middle_PIP_Joint: limit lower=0 upper=1.7453293 effort=3 velocity=10 -> lower=0 upper=0 effort=3 velocity=10
- joint R_Ring_ABAD_Joint: origin xyz=0.004401 0.0219725 -0.0476342 rpy=0.11155943312272709 -0.34233803538908836 -0.0870605140350752 -> xyz=0.004401 0.0219725 -0.0476342 rpy=0.111559433 -0.342338035 -0.087060514
- joint R_Ring_DIP_Joint: limit lower=0 upper=1.235693 effort=3 velocity=10 -> lower=0 upper=1.10975556 effort=0 velocity=0; mimic joint=R_Ring_PIP_Joint multiplier=0.6361 offset=0 -> joint=R_Ring_PIP_Joint multiplier=0.635843082 offset=0
- joint R_Ring_MCP_Joint: origin xyz=-0.003817 0 -0.0061246 rpy=0 0.3490658780677358 0 -> xyz=-0.003817 0 -0.0061246 rpy=0 0.349065878 0
- joint R_Ring_PIP_Joint: limit lower=0 upper=1.7453293 effort=3 velocity=10 -> lower=0 upper=0 effort=3 velocity=10
- joint R_Shoulder_Pitch_Joint: origin xyz=0 -0.0710988 0.0190509 rpy=-0.2617993931425453 -5.720983531354307e-08 2.6299670132234887e-06 -> xyz=0 -0.0710988 0.0190509 rpy=-0.261799393 -5.72098353e-08 2.62996701e-06
- joint R_Shoulder_Roll_Joint: origin xyz=-0.1365 -0.1195 0 rpy=0.2617993931425453 5.720983553558767e-08 2.6299670132234887e-06 -> xyz=-0.1365 -0.1195 0 rpy=0.261799393 5.72098355e-08 2.62996701e-06
- joint R_Thumb_CMC_Joint: origin xyz=0 -0.0139985 -0.0323434 rpy=0.268480430783685 0 0 -> xyz=0 -0.0139985 -0.0323434 rpy=0.268480431 0 0
- joint R_Thumb_IP_Joint: limit lower=0 upper=1.1397 effort=4.8 velocity=8 -> lower=0 upper=1.14964202 effort=0 velocity=0; mimic joint=R_Thumb_MCP_Joint multiplier=0.7319 offset=0 -> joint=R_Thumb_MCP_Joint multiplier=0.731884995 offset=0
- joint R_Thumb_Yaw_Joint: origin xyz=0.0330735 -0.0139336 0.0273021 rpy=-0.08570131975411865 0.12731092045638293 0.1266080083114749 -> xyz=0.0330735 -0.0139336 0.0273021 rpy=-0.0857013198 0.12731092 0.126608008
- joint Waist_Pitch_Dummy_Joint: limit lower=-0.523598 upper=0.785398 effort=126 velocity=8 -> lower=-0.523598 upper=0.785398 effort=0 velocity=0
- joint Waist_Upper_Pitch_Joint: limit lower=-0.785398 upper=0.523598 effort=126 velocity=8 -> lower=-0.785398 upper=0.523598 effort=0 velocity=0
- joint orbbec_color_optical_frame_joint: origin xyz=-0.002 -0.033 -0.001 rpy=0 1.5708 0 -> xyz=-0.002 -0.033 -0.001 rpy=-0 1.57079633 0
- joint orbbec_depth_optical_frame_joint: origin xyz=0 0 0 rpy=0 1.5708 0 -> xyz=0 0 0 rpy=-0 1.57079633 0
- joint realsense_color_optical_frame_joint: origin xyz=0.011 0.033 0.013 rpy=0 1.5708 0 -> xyz=0.011 0.033 0.013 rpy=-0 1.57079633 0
- joint realsense_depth_optical_frame_joint: origin xyz=0.011 0.018 0.013 rpy=0 1.5708 0 -> xyz=0.011 0.018 0.013 rpy=-0 1.57079633 0
- joint zed_left_camera_optical_frame_joint: origin xyz=0 0.032 0.013 rpy=0 1.5708 0 -> xyz=0 0.032 0.013 rpy=-0 1.57079633 0

Commit message: Republish proto_v2 from SSoT (LSQ couplings, updated inertials/friction)
emit_usd now authors LSQ-through-origin physxMimic/Newton couplings (matches
URDF); SSoT inertial/friction updates included; version-header comment dropped.
examples/ intentionally excluded (still under validation).

File: urdf/ALLEX.urdf (robot description, URDF)
Before this commit: robot ALLEX, 82 links, 81 joints
Links:
- link L_Forearm_Link: mass 3.02673929 -> 3.1
- link L_Upper_Arm_Link: mass 3.5 -> 3.51
- link L_Wrist_Pitch_Link: mass 1.1 -> 0.97383
- link L_Wrist_Roll_Link: mass 0.075462826 -> 0.172
- link R_Forearm_Link: mass 3.02673929 -> 3.1
- link R_Upper_Arm_Link: mass 3.5 -> 3.51
- link R_Wrist_Pitch_Link: mass 1.1 -> 0.97383
- link R_Wrist_Roll_Link: mass 0.075462826 -> 0.172
- link Waist_Upper_Pitch_Link: mass 3.24744786 -> 2.780295
