Commit message: Republish proto_v2: ROM/torque audit + MIT-mode examples (isaac, hello)
- mjcf/urdf/usd: ROM ranges and joint torque limits from the latest audit
  (hardware ROM doc + motor-datasheet peak); USD position limits are now
  single-sourced from the SSoT.
- examples: add isaac/replay.py (gravity-comp + PD) and hello.npz (a
  nominal-gain wave for PhysX, whose implicit drive lags demo1's low-gain
  compliant phases); refresh mujoco/replay.py and demo1.npz (dynamic gains,
  no dynamic torque limit); README documents MIT-mode (torque_ff + PD).
  The newton example is intentionally not published.

File: urdf/ALLEX.urdf (robot description, URDF)
Before this commit: robot ALLEX, 82 links, 81 joints
Joints:
- joint L_Index_ABAD_Joint: limit lower=-0.523599 upper=0.523599 effort=2.1 velocity=8 -> lower=-0.523599 upper=0.523599 effort=3.5 velocity=8
- joint L_Index_DIP_Joint: limit lower=0 upper=1.10975556 effort=3 velocity=10 -> lower=0 upper=1.25999882 effort=0 velocity=10; mimic joint=L_Index_PIP_Joint multiplier=0.635843082 offset=0 -> joint=L_Index_PIP_Joint multiplier=0.656296489 offset=0
- joint L_Index_MCP_Joint: limit lower=-0.174532 upper=1.570796 effort=4.8 velocity=8 -> lower=-0.174532 upper=1.570796 effort=5 velocity=8
- joint L_Index_PIP_Joint: limit lower=0 upper=1.7453293 effort=3 velocity=10 -> lower=0 upper=1.9198622 effort=3 velocity=10
- joint L_Little_ABAD_Joint: limit lower=-0.523599 upper=0.523599 effort=2.1 velocity=8 -> lower=-0.523599 upper=0.523599 effort=3.5 velocity=8
- joint L_Little_DIP_Joint: limit lower=0 upper=1.10975556 effort=3 velocity=10 -> lower=0 upper=1.25999882 effort=0 velocity=10; mimic joint=L_Little_PIP_Joint multiplier=0.635843082 offset=0 -> joint=L_Little_PIP_Joint multiplier=0.656296489 offset=0
- joint L_Little_MCP_Joint: limit lower=-0.174532 upper=1.570796 effort=4.8 velocity=8 -> lower=-0.174532 upper=1.570796 effort=5 velocity=8
- joint L_Little_PIP_Joint: limit lower=0 upper=1.7453293 effort=3 velocity=10 -> lower=0 upper=1.9198622 effort=3 velocity=10
- joint L_Middle_ABAD_Joint: limit lower=-0.523599 upper=0.523599 effort=2.1 velocity=8 -> lower=-0.523599 upper=0.523599 effort=3.5 velocity=8
- joint L_Middle_DIP_Joint: limit lower=0 upper=1.10975556 effort=3 velocity=10 -> lower=0 upper=1.25999882 effort=0 velocity=10; mimic joint=L_Middle_PIP_Joint multiplier=0.635843082 offset=0 -> joint=L_Middle_PIP_Joint multiplier=0.656296489 offset=0
- joint L_Middle_MCP_Joint: limit lower=-0.174532 upper=1.570796 effort=4.8 velocity=8 -> lower=-0.174532 upper=1.570796 effort=5 velocity=8
- joint L_Middle_PIP_Joint: limit lower=0 upper=1.7453293 effort=3 velocity=10 -> lower=0 upper=1.9198622 effort=3 velocity=10
- joint L_Ring_ABAD_Joint: limit lower=-0.523599 upper=0.523599 effort=2.1 velocity=8 -> lower=-0.523599 upper=0.523599 effort=3.5 velocity=8
- joint L_Ring_DIP_Joint: limit lower=0 upper=1.10975556 effort=3 velocity=10 -> lower=0 upper=1.25999882 effort=0 velocity=10; mimic joint=L_Ring_PIP_Joint multiplier=0.635843082 offset=0 -> joint=L_Ring_PIP_Joint multiplier=0.656296489 offset=0
- joint L_Ring_MCP_Joint: limit lower=-0.174532 upper=1.570796 effort=4.8 velocity=8 -> lower=-0.174532 upper=1.570796 effort=5 velocity=8
- joint L_Ring_PIP_Joint: limit lower=0 upper=1.7453293 effort=3 velocity=10 -> lower=0 upper=1.9198622 effort=3 velocity=10
- joint L_Thumb_CMC_Joint: limit lower=0 upper=1.570796 effort=4.8 velocity=8 -> lower=0 upper=1.570796 effort=4.5 velocity=8
- joint L_Thumb_IP_Joint: limit lower=0 upper=1.14964202 effort=4.8 velocity=8 -> lower=0 upper=1.14964202 effort=0 velocity=8
- joint L_Thumb_MCP_Joint: limit lower=0 upper=1.570796 effort=4.8 velocity=8 -> lower=0 upper=1.570796 effort=3 velocity=8
- joint L_Thumb_Yaw_Joint: limit lower=0 upper=2.617994 effort=2.9 velocity=5 -> lower=0 upper=2.617994 effort=1.5 velocity=5
- joint L_Wrist_Pitch_Joint: limit lower=-1.396263 upper=1.396263 effort=45 velocity=30 -> lower=-1.396263 upper=1.396263 effort=18 velocity=30
- joint L_Wrist_Roll_Joint: limit lower=-0.872665 upper=0.872665 effort=45 velocity=30 -> lower=-0.872665 upper=0.872665 effort=20 velocity=30
- joint Neck_Pitch_Joint: limit lower=-0.523599 upper=0.785398 effort=12 velocity=20 -> lower=-0.6981317 upper=0.8726646 effort=12 velocity=20
- joint R_Elbow_Joint: limit lower=-2.879793 upper=0.087266 effort=100 velocity=20 -> lower=-2.7925268 upper=0.0872665 effort=100 velocity=20
- joint R_Index_ABAD_Joint: limit lower=-0.523599 upper=0.523599 effort=2.1 velocity=8 -> lower=-0.523599 upper=0.523599 effort=3.5 velocity=8
- joint R_Index_DIP_Joint: limit lower=0 upper=1.10975556 effort=3 velocity=10 -> lower=0 upper=1.25999882 effort=0 velocity=10; mimic joint=R_Index_PIP_Joint multiplier=0.635843082 offset=0 -> joint=R_Index_PIP_Joint multiplier=0.656296489 offset=0
- joint R_Index_MCP_Joint: limit lower=-0.174532 upper=1.570796 effort=4.8 velocity=8 -> lower=-0.174532 upper=1.570796 effort=5 velocity=8
- joint R_Index_PIP_Joint: limit lower=0 upper=1.7453293 effort=3 velocity=10 -> lower=0 upper=1.9198622 effort=3 velocity=10
- joint R_Little_ABAD_Joint: limit lower=-0.523599 upper=0.523599 effort=2.1 velocity=8 -> lower=-0.523599 upper=0.523599 effort=3.5 velocity=8
- joint R_Little_DIP_Joint: limit lower=0 upper=1.10975556 effort=3 velocity=10 -> lower=0 upper=1.25999882 effort=0 velocity=10; mimic joint=R_Little_PIP_Joint multiplier=0.635843082 offset=0 -> joint=R_Little_PIP_Joint multiplier=0.656296489 offset=0
- joint R_Little_MCP_Joint: limit lower=-0.174532 upper=1.570796 effort=4.8 velocity=8 -> lower=-0.174532 upper=1.570796 effort=5 velocity=8
- joint R_Little_PIP_Joint: limit lower=0 upper=1.7453293 effort=3 velocity=10 -> lower=0 upper=1.9198622 effort=3 velocity=10
- joint R_Middle_ABAD_Joint: limit lower=-0.523599 upper=0.523599 effort=2.1 velocity=8 -> lower=-0.523599 upper=0.523599 effort=3.5 velocity=8
- joint R_Middle_DIP_Joint: limit lower=0 upper=1.10975556 effort=3 velocity=10 -> lower=0 upper=1.25999882 effort=0 velocity=10; mimic joint=R_Middle_PIP_Joint multiplier=0.635843082 offset=0 -> joint=R_Middle_PIP_Joint multiplier=0.656296489 offset=0
- joint R_Middle_MCP_Joint: limit lower=-0.174532 upper=1.570796 effort=4.8 velocity=8 -> lower=-0.174532 upper=1.570796 effort=5 velocity=8
- joint R_Middle_PIP_Joint: limit lower=0 upper=1.7453293 effort=3 velocity=10 -> lower=0 upper=1.9198622 effort=3 velocity=10
- joint R_Ring_ABAD_Joint: limit lower=-0.523599 upper=0.523599 effort=2.1 velocity=8 -> lower=-0.523599 upper=0.523599 effort=3.5 velocity=8
- joint R_Ring_DIP_Joint: limit lower=0 upper=1.10975556 effort=3 velocity=10 -> lower=0 upper=1.25999882 effort=0 velocity=10; mimic joint=R_Ring_PIP_Joint multiplier=0.635843082 offset=0 -> joint=R_Ring_PIP_Joint multiplier=0.656296489 offset=0
- joint R_Ring_MCP_Joint: limit lower=-0.174532 upper=1.570796 effort=4.8 velocity=8 -> lower=-0.174532 upper=1.570796 effort=5 velocity=8
- joint R_Ring_PIP_Joint: limit lower=0 upper=1.7453293 effort=3 velocity=10 -> lower=0 upper=1.9198622 effort=3 velocity=10
- joint R_Thumb_CMC_Joint: limit lower=0 upper=1.570796 effort=4.8 velocity=8 -> lower=0 upper=1.570796 effort=4.5 velocity=8
- joint R_Thumb_IP_Joint: limit lower=0 upper=1.14964202 effort=4.8 velocity=8 -> lower=0 upper=1.14964202 effort=0 velocity=8
- joint R_Thumb_MCP_Joint: limit lower=0 upper=1.570796 effort=4.8 velocity=8 -> lower=0 upper=1.570796 effort=3 velocity=8
- joint R_Thumb_Yaw_Joint: limit lower=-2.617994 upper=0 effort=2.9 velocity=5 -> lower=-2.617994 upper=0 effort=1.5 velocity=5
- joint R_Wrist_Pitch_Joint: limit lower=-1.396263 upper=1.396263 effort=45 velocity=30 -> lower=-1.396263 upper=1.396263 effort=18 velocity=30
- joint R_Wrist_Roll_Joint: limit lower=-0.872665 upper=0.872665 effort=45 velocity=30 -> lower=-0.872665 upper=0.872665 effort=20 velocity=30
- joint Waist_Lower_Pitch_Joint: limit lower=-0.523598 upper=0.785398 effort=126 velocity=8 -> lower=-0.5235988 upper=1.0471976 effort=152 velocity=8
- joint Waist_Pitch_Dummy_Joint: limit lower=-0.523598 upper=0.785398 effort=126 velocity=8 -> lower=-0.5235988 upper=1.0471976 effort=0 velocity=8
- joint Waist_Upper_Pitch_Joint: limit lower=-0.785398 upper=0.523598 effort=126 velocity=8 -> lower=-1.0471976 upper=0.5235988 effort=0 velocity=8
- joint Waist_Yaw_Joint: limit lower=-2.792526 upper=2.792526 effort=126 velocity=8 -> lower=-2.8797933 upper=2.8797933 effort=130 velocity=8
